File: MCU.sch (KiCad schematic (older format))
At the start: 0 parts

Commit message: Trabajo dia 1, micro organizado
Parts:
- added C? (x3): 0.1u, symbol Device:C
- added C?: 22u, symbol Device:CP
- added J?: UART/PROG, symbol Connector_Generic:Conn_01x04
- added JP?: BOOT, symbol Device:Jumper
- added R?: 1k, symbol Device:R
- added SW?: SW_Push, symbol Switch:SW_Push
- added U?: ESP32-WROOM-32D, RF_Module:ESP32-WROOM-32, symbol RF_Module:ESP32-WROOM-32D
Connections:
- new net +3V3: C?.1, C?.1, J?.1 (Pin_1), R?.1, U?.2 (VDD)
- new net ADC-ALERT: U?.6 (IO34)
- new net BCCU: U?.12 (IO27)
- new net BOOT: JP?.1, U?.25 (IO0)
- new net BTN_0: U?.27 (IO16)
- new net BTN_1: U?.23 (IO15)
- new net BTN_2: U?.13 (IO14)
- new net BTN_3: U?.16 (IO13)
- new net FAN: U?.28 (IO17)
- new net GND: C?.1, C?.2, C?.2, C?.2, J?.2 (Pin_2), JP?.2, SW?.2, U?.1 (GND), U?.15 (GND), U?.38 (GND), U?.39 (GND)
- new net IR2104-EN: U?.8 (IO32)
- new net MISO: U?.31 (IO19)
- new net MOSI: U?.37 (IO23)
- new net NTC_BAT: U?.10 (IO25)
- new net NTC_DIS: U?.7 (IO35)
- new net RST_MCU: C?.1, C?.2, R?.2, SW?.1, U?.3 (EN)
- new net SCK: U?.30 (IO18)
- new net SCL: U?.36 (IO22)
- new net SDA: U?.33 (IO21)
- new net UART_RX: J?.3 (Pin_3), U?.34 (RXD0/IO3)
- new net UART_TX: J?.4 (Pin_4), U?.35 (TXD0/IO1)
- new net ~SS0: U?.29 (IO5)
- no-connect marks 0 -> 13
Other:
- note added: "CONTROL"
- note added: "HEADERS"
- note added: "I2C"
- note added: "INTERFAZ"
- note added: "IO PORTS"
- note added: "MCU"
- note added: "MPPT"
- note added: "PERIFERICOS"
- note added: "RESET"
- note added: "SPI"
- note added: "TERMICO"
- note added: "UART\n"
