File: MCU.sch (KiCad schematic (older format))
At the start: 9 parts

Commit message: Actualizado 15/10
Parts:
- R?: value 1k -> 10k
Changed lines of the file:
@@
 $Descr A4 11693 8268
 encoding utf-8
-Sheet 2 7
+Sheet 2 8
 Title "Microcontrolador principal"
 Date "2021-10-11"
@@
 P 4900 2500
 F 0 "R?" H 4970 2546 50  0000 L CNN
-F 1 "1k" H 4970 2455 50  0000 L CNN
+F 1 "10k" H 4970 2455 50  0000 L CNN
 F 2 "" V 4830 2500 50  0001 C CNN
 F 3 "~" H 4900 2500 50  0001 C CNN

Commit message: Esquemático acabado y asignación de huellas
Parts:
- C1, C2, C4: renamed from C?; footprint (none) -> Capacitors_SMD:C_0603
- C3: renamed from C?; footprint (none) -> Capacitors_SMD:CP_Elec_5x4.5
- J1: renamed from J?; footprint (none) -> Pin_Headers:Pin_Header_Straight_1x04_Pitch2.54mm
- JP1: renamed from JP?; footprint (none) -> Pin_Headers:Pin_Header_Straight_1x02_Pitch2.54mm
- R1: renamed from R?; footprint (none) -> Resistors_SMD:R_0603
- SW1: renamed from SW?; footprint (none) -> Buttons_Switches_SMD:SW_SPST_B3U-1000P
- U1: renamed from U?; footprint RF_Module:ESP32-WROOM-32 -> ESP32-footprints-Lib:ESP32-WROOM
Connections:
- net UART_INT: now reaches U1.14 (IO12)
- no-connect marks 13 -> 12
Changed lines of the file:
@@
 $EndDescr
 $Comp
-L RF_Module:ESP32-WROOM-32D U?
+L RF_Module:ESP32-WROOM-32D U1
 U 1 1 616452B2
 P 6050 4050
-F 0 "U?" H 5650 2650 50  0000 C CNN
+F 0 "U1" H 5650 2650 50  0000 C CNN
 F 1 "ESP32-WROOM-32D" H 6550 2650 50  0000 C CNN
-F 2 "RF_Module:ESP32-WROOM-32" H 6050 2550 50  0001 C CNN
+F 2 "ESP32-footprints-Lib:ESP32-WROOM" H 6050 2550 50  0001 C CNN
 F 3 "https://www.espressif.com/sites/default/files/documentation/esp32-wroom-32d_esp32-wroom-32u_datasheet_en.pdf" H 5750 4100 50  0001 C CNN
 	1    6050 4050
@@
 IO_3
 Wire Wire Line
-	9900 1350 9550 1350
-Wire Wire Line
-	9900 1550 9550 1550
-Text Label 9550 1350 0    50   ~ 0
+	9900 1200 9550 1200
+Wire Wire Line
+	9900 1400 9550 1400
+Text Label 9550 1200 0    50   ~ 0
 IO_1
-Text Label 9550 1550 0    50   ~ 0
+Text Label 9550 1400 0    50   ~ 0
 IO_3
-Text GLabel 9900 1350 2    50   Output ~ 0
+Text GLabel 9900 1200 2    50   Output ~ 0
 UART_TX
-Text GLabel 9900 1550 2    50   Input ~ 0
+Text GLabel 9900 1400 2    50   Input ~ 0
 UART_RX
 $Comp
-L power:+3.3V #PWR?
+L power:+3.3V #PWR07
 U 1 1 61648D95
 P 6050 1950
-F 0 "#PWR?" H 6050 1800 50  0001 C CNN
+F 0 "#PWR07" H 6050 1800 50  0001 C CNN
 F 1 "+3.3V" H 6065 2123 50  0000 C CNN
 F 2 "" H 6050 1950 50  0001 C CNN
@@
 Wire Wire Line
 	10050 3400 9600 3400
-Text Notes 9800 1150 0    50   ~ 0
+Text Notes 9800 1000 0    50   ~ 0
 UART\n
 Text Notes 9850 2600 0    50   ~ 0
@@
 BOOT
 $Comp
-L Device:Jumper JP?
+L Device:Jumper JP1
 U 1 1 6167B7F0
 P 1900 5600
-F 0 "JP?" H 1900 5864 50  0000 C CNN
+F 0 "JP1" H 1900 5864 50  0000 C CNN
 F 1 "BOOT" H 1900 5773 50  0000 C CNN
-F 2 "" H 1900 5600 50  0001 C CNN
+F 2 "Pin_Headers:Pin_Header_Straight_1x02_Pitch2.54mm" H 1900 5600 50  0001 C CNN
 F 3 "~" H 1900 5600 50  0001 C CNN
 	1    1900 5600
@@
 	1600 5600 1450 5600
 $Comp
-L power:GND #PWR?
+L power:GND #PWR04
 U 1 1 6167D748
 P 2500 5800
-F 0 "#PWR?" H 2500 5550 50  0001 C CNN
+F 0 "#PWR04" H 2500 5550 50  0001 C CNN
 F 1 "GND" H 2505 5627 50  0000 C CNN
 F 2 "" H 2500 5800 50  0001 C CNN
@@
 	2500 5600 2200 5600
 $Comp
-L Switch:SW_Push SW?
+L Switch:SW_Push SW1
 U 1 1 61680338
 P 1950 4050
-F 0 "SW?" H 1950 4335 50  0000 C CNN
+F 0 "SW1" H 1950 4335 50  0000 C CNN
 F 1 "SW_Push" H 1950 4244 50  0000 C CNN
-F 2 "" H 1950 4250 50  0001 C CNN
+F 2 "Buttons_Switches_SMD:SW_SPST_B3U-1000P" H 1950 4250 50  0001 C CNN
 F 3 "~" H 1950 4250 50  0001 C CNN
 	1    1950 4050
@@
 RST_MCU
 $Comp
-L Device:C C?
+L Device:C C1
 U 1 1 6168224F
 P 1950 4300
-F 0 "C?" V 2202 4300 50  0000 C CNN
+F 0 "C1" V 2202 4300 50  0000 C CNN
 F 1 "0.1u" V 2111 4300 50  0000 C CNN
-F 2 "" H 1988 4150 50  0001 C CNN
+F 2 "Capacitors_SMD:C_0603" H 1988 4150 50  0001 C CNN
 F 3 "~" H 1950 4300 50  0001 C CNN
 	1    1950 4300
@@
 Connection ~ 2300 4050
 $Comp
-L power:GND #PWR?
+L power:GND #PWR03
 U 1 1 61693D9B
 P 2500 4400
-F 0 "#PWR?" H 2500 4150 50  0001 C CNN
+F 0 "#PWR03" H 2500 4150 50  0001 C CNN
 F 1 "GND" H 2505 4227 50  0000 C CNN
 F 2 "" H 2500 4400 50  0001 C CNN
@@
 	2500 4050 2500 4400
 $Comp
-L Connector_Generic:Conn_01x04 J?
+L Connector_Generic:Conn_01x04 J1
 U 1 1 616975FB
 P 2450 6750
-F 0 "J?" H 2530 6742 50  0000 L CNN
+F 0 "J1" H 2530 6742 50  0000 L CNN
 F 1 "UART/PROG" H 2530 6651 50  0000 L CNN
-F 2 "" H 2450 6750 50  0001 C CNN
+F 2 "Pin_Headers:Pin_Header_Straight_1x04_Pitch2.54mm" H 2450 6750 50  0001 C CNN
 F 3 "~" H 2450 6750 50  0001 C CNN
 	1    2450 6750
@@
 $EndComp
 $Comp
-L power:+3.3V #PWR?
+L power:+3.3V #PWR01
 U 1 1 6169942A
 P 1600 6600
-F 0 "#PWR?" H 1600 6450 50  0001 C CNN
+F 0 "#PWR01" H 1600 6450 50  0001 C CNN
 F 1 "+3.3V" H 1615 6773 50  0000 C CNN
 F 2 "" H 1600 6600 50  0001 C CNN
@@
 $EndComp
 $Comp
-L power:GND #PWR?
+L power:GND #PWR02
 U 1 1 6169B60B
 P 1600 6800
-F 0 "#PWR?" H 1600 6550 50  0001 C CNN
+F 0 "#PWR02" H 1600 6550 50  0001 C CNN
 F 1 "GND" H 1605 6627 50  0000 C CNN
 F 2 "" H 1600 6800 50  0001 C CNN
@@
 	1600 6750 1600 6800
 $Comp
-L Device:R R?
+L Device:R R1
 U 1 1 616BC8FE
 P 4900 2500
-F 0 "R?" H 4970 2546 50  0000 L CNN
+F 0 "R1" H 4970 2546 50  0000 L CNN
 F 1 "10k" H 4970 2455 50  0000 L CNN
-F 2 "" V 4830 2500 50  0001 C CNN
+F 2 "Resistors_SMD:R_0603" V 4830 2500 50  0001 C CNN
 F 3 "~" H 4900 2500 50  0001 C CNN
 	1    4900 2500
@@
 $EndComp
 $Comp
-L Device:C C?
+L Device:C C2
 U 1 1 616BD15F
 P 4900 3100
-F 0 "C?" H 5015 3146 50  0000 L CNN
+F 0 "C2" H 5015 3146 50  0000 L CNN
 F 1 "0.1u" H 5015 3055 50  0000 L CNN
-F 2 "" H 4938 2950 50  0001 C CNN
+F 2 "Capacitors_SMD:C_0603" H 4938 2950 50  0001 C CNN
 F 3 "~" H 4900 3100 50  0001 C CNN
 	1    4900 3100
@@
 $EndComp
 $Comp
-L power:+3.3V #PWR?
+L power:+3.3V #PWR05
 U 1 1 616BD52D
 P 4900 2150
-F 0 "#PWR?" H 4900 2000 50  0001 C CNN
+F 0 "#PWR05" H 4900 2000 50  0001 C CNN
 F 1 "+3.3V" H 4915 2323 50  0000 C CNN
 F 2 "" H 4900 2150 50  0001 C CNN
@@
 	4900 2950 4900 2850
 $Comp
-L power:GND #PWR?
+L power:GND #PWR06
 U 1 1 616C50B6
 P 4900 3550
-F 0 "#PWR?" H 4900 3300 50  0001 C CNN
+F 0 "#PWR06" H 4900 3300 50  0001 C CNN
 F 1 "GND" H 4905 3377 50  0000 C CNN
 F 2 "" H 4900 3550 50  0001 C CNN
@@
 	4900 3250 4900 3550
 $Comp
-L Device:C C?
+L Device:C C4
 U 1 1 616CDD2F
 P 6700 2200
-F 0 "C?" H 6815 2246 50  0000 L CNN
+F 0 "C4" H 6815 2246 50  0000 L CNN
 F 1 "0.1u" H 6815 2155 50  0000 L CNN
-F 2 "" H 6738 2050 50  0001 C CNN
+F 2 "Capacitors_SMD:C_0603" H 6738 2050 50  0001 C CNN
 F 3 "~" H 6700 2200 50  0001 C CNN
 	1    6700 2200
@@
 $EndComp
 $Comp
-L Device:CP C?
+L Device:CP C3
 U 1 1 616CE25D
 P 6300 2200
-F 0 "C?" H 6418 2246 50  0000 L CNN
+F 0 "C3" H 6418 2246 50  0000 L CNN
 F 1 "22u" H 6418 2155 50  0000 L CNN
-F 2 "" H 6338 2050 50  0001 C CNN
+F 2 "Capacitors_SMD:CP_Elec_5x4.5" H 6338 2050 50  0001 C CNN
 F 3 "~" H 6300 2200 50  0001 C CNN
 	1    6300 2200
@@
 	6300 2400 6300 2350
 $Comp
-L power:GND #PWR?
+L power:GND #PWR08
 U 1 1 61648625
 P 6050 5600
-F 0 "#PWR?" H 6050 5350 50  0001 C CNN
+F 0 "#PWR08" H 6050 5350 50  0001 C CNN
 F 1 "GND" H 6055 5427 50  0000 C CNN
 F 2 "" H 6050 5600 50  0001 C CNN
@@
 $EndComp
 $Comp
-L power:GND #PWR?
+L power:GND #PWR09
 U 1 1 616DF7B7
 P 6500 2500
-F 0 "#PWR?" H 6500 2250 50  0001 C CNN
+F 0 "#PWR09" H 6500 2250 50  0001 C CNN
 F 1 "GND" H 6505 2327 50  0000 C CNN
 F 2 "" H 6500 2500 50  0001 C CNN
@@
 PERIFERICOS
 Wire Notes Line
-	9400 3550 9400 1050
+	9400 3550 9400 900
 Wire Notes Line
 	9400 4550 9400 3800
@@
 NoConn ~ 6650 3050
 NoConn ~ 6650 3250
-NoConn ~ 6650 3450
+NoConn ~ 6650 4950
 NoConn ~ 6650 4650
-NoConn ~ 6650 4950
+Wire Wire Line
+	6650 3450 6950 3450
+Text Label 6950 3450 2    50   ~ 0
+IO_12
+Wire Wire Line
+	9900 1600 9550 1600
+Text Label 9550 1600 0    50   ~ 0
+IO_12
+Text GLabel 9900 1600 2    50   Input ~ 0
+UART_INT
 $EndSCHEMATC
