File: proyectoSolar.sch (KiCad schematic (older format))
At the start: 0 parts

Commit message: Trabajo dia 1, micro organizado
Changed lines of the file:
@@
 $Descr A4 11693 8268
 encoding utf-8
-Sheet 1 5
+Sheet 1 7
 Title ""
 Date ""
@@
 $EndDescr
 $Sheet
-S 1600 1150 1650 1400
+S 2400 1800 1650 1400
 U 61644852
 F0 "MCU" 50
@@
 $EndSheet
 $Sheet
-S 3850 1150 1900 1400
+S 4650 1800 1900 1400
 U 61644BD1
 F0 "power" 50
@@
 $EndSheet
 $Sheet
-S 6700 1150 2050 1350
+S 7500 1800 2050 1350
 U 61644C06
 F0 "MPPT" 50
@@
 $EndSheet
 $Sheet
-S 2700 3450 1750 1000
+S 1750 4100 1750 1000
 U 61644C46
 F0 "thermo" 50
@@
 $EndSheet
 $Sheet
-S 5300 3450 1900 1000
+S 4350 4100 1900 1000
 U 61644CA5
 F0 "inverter" 50
 F1 "inverter.sch" 50
 $EndSheet
+$Sheet
+S 7600 4100 2200 1100
+U 6167B4C8
+F0 "interfaz" 50
+F1 "interfaz.sch" 50
+$EndSheet
 $EndSCHEMATC

Commit message: Actualizado 15/10
Changed lines of the file:
@@
 $Descr A4 11693 8268
 encoding utf-8
-Sheet 1 7
+Sheet 1 8
 Title ""
 Date ""
@@
 $EndDescr
 $Sheet
-S 2400 1800 1650 1400
+S 7000 3800 1900 1400
 U 61644852
 F0 "MCU" 50
@@
 $EndSheet
 $Sheet
-S 4650 1800 1900 1400
+S 2900 2150 1900 1400
 U 61644BD1
 F0 "power" 50
@@
 $EndSheet
 $Sheet
-S 7500 1800 2050 1350
+S 4950 2150 1900 1400
 U 61644C06
 F0 "MPPT" 50
@@
 $EndSheet
 $Sheet
-S 1750 4100 1750 1000
-U 61644C46
-F0 "thermo" 50
-F1 "thermo.sch" 50
-$EndSheet
-$Sheet
-S 4350 4100 1900 1000
+S 7000 2150 1900 1400
 U 61644CA5
 F0 "inverter" 50
@@
 $EndSheet
 $Sheet
-S 7600 4100 2200 1100
+S 4950 3800 1900 1400
 U 6167B4C8
 F0 "interfaz" 50
 F1 "interfaz.sch" 50
 $EndSheet
+$Sheet
+S 2900 3800 1900 1400
+U 61644C46
+F0 "monitor" 50
+F1 "monitor.sch" 50
+$EndSheet
 $EndSCHEMATC
