File: monitor.sch (KiCad schematic (older format))
At the start: 3 parts

Commit message: Esquemático acabado y asignación de huellas
Parts:
- C29: renamed from C?; footprint (none) -> Capacitors_SMD:C_0603
- R41: renamed from R?; value R -> 10k; footprint (none) -> Resistors_SMD:R_0603
- U7: renamed from U?; footprint Package_SO:TSSOP-10_3x3mm_P0.5mm -> Housings_SSOP:MSOP-10_3x3mm_Pitch0.5mm
Changed lines of the file:
@@
 $EndDescr
 $Comp
-L Analog_ADC:ADS1015IDGS U?
+L Analog_ADC:ADS1015IDGS U7
 U 1 1 616A8659
 P 5550 3650
-F 0 "U?" H 5200 4200 50  0000 C CNN
+F 0 "U7" H 5200 4200 50  0000 C CNN
 F 1 "ADS1015IDGS" H 5150 4100 50  0000 C CNN
-F 2 "Package_SO:TSSOP-10_3x3mm_P0.5mm" H 5550 3150 50  0001 C CNN
+F 2 "Housings_SSOP:MSOP-10_3x3mm_Pitch0.5mm" H 5550 3150 50  0001 C CNN
 F 3 "http://www.ti.com/lit/ds/symlink/ads1015.pdf" H 5500 2750 50  0001 C CNN
 	1    5550 3650
@@
 $EndComp
 $Comp
-L Device:C C?
+L Device:C C29
 U 1 1 616A97E2
 P 6350 4100
-F 0 "C?" V 6098 4100 50  0000 C CNN
+F 0 "C29" V 6098 4100 50  0000 C CNN
 F 1 "100nF" V 6189 4100 50  0000 C CNN
-F 2 "" H 6388 3950 50  0001 C CNN
+F 2 "Capacitors_SMD:C_0603" H 6388 3950 50  0001 C CNN
 F 3 "~" H 6350 4100 50  0001 C CNN
 	1    6350 4100
@@
 $EndComp
 $Comp
-L power:+3.3V #PWR?
+L power:+3.3V #PWR043
 U 1 1 616AB32D
 P 6800 3000
-F 0 "#PWR?" H 6800 2850 50  0001 C CNN
+F 0 "#PWR043" H 6800 2850 50  0001 C CNN
 F 1 "+3.3V" V 6815 3128 50  0000 L CNN
 F 2 "" H 6800 3000 50  0001 C CNN
@@
 $EndComp
 $Comp
-L power:GND #PWR?
+L power:GND #PWR042
 U 1 1 616AB99C
 P 5550 4200
-F 0 "#PWR?" H 5550 3950 50  0001 C CNN
+F 0 "#PWR042" H 5550 3950 50  0001 C CNN
 F 1 "GND" H 5555 4027 50  0000 C CNN
 F 2 "" H 5550 4200 50  0001 C CNN
@@
 	5000 3850 5150 3850
 $Comp
-L Device:R R?
+L Device:R R41
 U 1 1 616AEC49
 P 6250 3300
-F 0 "R?" V 6043 3300 50  0000 C CNN
-F 1 "R" V 6134 3300 50  0000 C CNN
-F 2 "" V 6180 3300 50  0001 C CNN
+F 0 "R41" V 6043 3300 50  0000 C CNN
+F 1 "10k" V 6134 3300 50  0000 C CNN
+F 2 "Resistors_SMD:R_0603" V 6180 3300 50  0001 C CNN
 F 3 "~" H 6250 3300 50  0001 C CNN
 	1    6250 3300
