File: power.sch (KiCad schematic (older format))
At the start: 0 parts

Commit message: Trabajo de Carmen y Javi
Parts:
- added C14, C16: 100uF, symbol Device:CP
- added C15, C17: 33nF, symbol Device:C
- added C18: 47uF, symbol Device:CP
- added C5, C6: 4.7uF, symbol Device:CP
- added D5, D6: 5S310, symbol Device:D_Schottky
- added L2, L3: 100uH, symbol Device:L
- added R14, R15: 15k, symbol Device:R
- added R16: 1k, symbol Device:R
- added R17, R18: 33k, symbol Device:R
- added R19: 10k, symbol Device:R
- added U5, U6: XL7005A, symbol Device:XL7005A
- added U?: AMS1117-5.0, Package_TO_SOT_SMD:SOT-223-3_TabPin2, symbol Regulator_Linear:AMS1117-5.0
Connections:
- net labels added: +12V, +3.3V, +5V, GND, XL7005A-VIN
- wire segments 0 -> 100
