File: power.sch (KiCad schematic (older format))
At the start: 20 parts, among them U5 XL7005A, U6 XL7005A

Commit message: Actualizada y arreglada librería de componentes
Parts:
- U5, U6: symbol Device:XL7005A -> Local:XL7005A
Connections:
- wire segments 100 -> 96
Changed lines of the file:
@@
 	5200 4400 5600 4400
 $Comp
-L Device:XL7005A U5
+L Local:XL7005A U5
 U 1 1 616E3EAE
 P 3800 4250
@@
 	5100 2650 5100 2800
 $Comp
-L Device:XL7005A U6
+L Local:XL7005A U6
 U 1 1 6171D115
 P 3950 2700
@@
 	4300 3300 4300 2950
 Connection ~ 4600 3300
-Wire Wire Line
-	3450 4050 3450 4200
 Connection ~ 3450 4950
 Wire Wire Line
 	3450 4950 4200 4950
-Connection ~ 3450 4200
-Wire Wire Line
-	3450 4200 3450 4350
-Connection ~ 3450 4350
-Wire Wire Line
-	3450 4350 3450 4500
-Connection ~ 3450 4500
-Wire Wire Line
-	3450 4500 3450 4950
-Wire Wire Line
-	3450 4050 3450 3300
 Wire Wire Line
 	3450 2500 3600 2500
-Connection ~ 3450 4050
 Wire Wire Line
 	3600 2650 3450 2650
@@
 	6600 2300 8550 2300
 Connection ~ 6600 2300
+Wire Wire Line
+	3450 3300 3450 4950
 $EndSCHEMATC

Commit message: Esquemático acabado y asignación de huellas
Parts:
- C10: renamed from C5; footprint (none) -> Capacitors_SMD:CP_Elec_3x5.3
- C11: renamed from C6; footprint (none) -> Capacitors_SMD:CP_Elec_3x5.3
- C5: renamed from C18; footprint (none) -> Capacitors_SMD:CP_Elec_5x4.5
- C6: renamed from C17; footprint (none) -> Capacitors_SMD:C_0603
- C7: renamed from C15; footprint (none) -> Capacitors_SMD:C_0603
- C8: renamed from C16; footprint (none) -> Capacitors_SMD:CP_Elec_5x4.5
- C9: renamed from C14; footprint (none) -> Capacitors_SMD:CP_Elec_5x4.5
- D1: renamed from D5; footprint (none) -> Diodes_SMD:D_SOD-123
- D2: renamed from D6; footprint (none) -> Diodes_SMD:D_SOD-123
- L1: renamed from L3; footprint (none) -> Inductors_SMD:L_7.3x7.3_H3.5
- L2: footprint (none) -> Inductors_SMD:L_7.3x7.3_H3.5
- R2: renamed from R17; footprint (none) -> Resistors_SMD:R_0603
- R3: renamed from R19; footprint (none) -> Resistors_SMD:R_0603
- R4: renamed from R14; footprint (none) -> Resistors_SMD:R_0603
- R5: renamed from R16; footprint (none) -> Resistors_SMD:R_0603
- R6: renamed from R18; footprint (none) -> Resistors_SMD:R_0603
- R7: renamed from R15; footprint (none) -> Resistors_SMD:R_0603
- U2: renamed from U5; footprint (none) -> Housings_SOIC:SOIC-8-1EP_3.9x4.9mm_Pitch1.27mm
- U3: renamed from U6; footprint (none) -> Housings_SOIC:SOIC-8-1EP_3.9x4.9mm_Pitch1.27mm
- U4: renamed from U?; footprint Package_TO_SOT_SMD:SOT-223-3_TabPin2 -> TO_SOT_Packages_SMD:SOT-223-3_TabPin2
Connections:
- net GND: now also U2.5 (GND), U2.6 (GND), U2.7 (GND), U2.8 (GND)
Changed lines of the file:
@@
 $EndDescr
 $Comp
-L Device:R R16
+L Device:R R5
 U 1 1 616C27E8
 P 5600 4700
-F 0 "R16" H 5670 4746 50  0000 L CNN
+F 0 "R5" H 5670 4746 50  0000 L CNN
 F 1 "1k" H 5670 4655 50  0000 L CNN
-F 2 "" V 5530 4700 50  0001 C CNN
+F 2 "Resistors_SMD:R_0603" V 5530 4700 50  0001 C CNN
 F 3 "~" H 5600 4700 50  0001 C CNN
 	1    5600 4700
@@
 $EndComp
 $Comp
-L Device:R R14
+L Device:R R4
 U 1 1 616C319C
 P 5600 4100
-F 0 "R14" H 5670 4146 50  0000 L CNN
+F 0 "R4" H 5670 4146 50  0000 L CNN
 F 1 "15k" H 5670 4055 50  0000 L CNN
-F 2 "" V 5530 4100 50  0001 C CNN
+F 2 "Resistors_SMD:R_0603" V 5530 4100 50  0001 C CNN
 F 3 "~" H 5600 4100 50  0001 C CNN
 	1    5600 4100
@@
 $EndComp
 $Comp
-L Device:R R15
+L Device:R R7
 U 1 1 616C3E27
 P 6050 4100
-F 0 "R15" H 6120 4146 50  0000 L CNN
+F 0 "R7" H 6120 4146 50  0000 L CNN
 F 1 "15k" H 6120 4055 50  0000 L CNN
-F 2 "" V 5980 4100 50  0001 C CNN
+F 2 "Resistors_SMD:R_0603" V 5980 4100 50  0001 C CNN
 F 3 "~" H 6050 4100 50  0001 C CNN
 	1    6050 4100
@@
 $EndComp
 $Comp
-L Device:R R19
+L Device:R R3
 U 1 1 616C43C2
 P 5600 3150
-F 0 "R19" H 5670 3196 50  0000 L CNN
+F 0 "R3" H 5670 3196 50  0000 L CNN
 F 1 "10k" H 5670 3105 50  0000 L CNN
-F 2 "" V 5530 3150 50  0001 C CNN
+F 2 "Resistors_SMD:R_0603" V 5530 3150 50  0001 C CNN
 F 3 "~" H 5600 3150 50  0001 C CNN
 	1    5600 3150
@@
 $EndComp
 $Comp
-L Device:R R17
+L Device:R R2
 U 1 1 616C4AE6
 P 5600 2500
-F 0 "R17" H 5670 2546 50  0000 L CNN
+F 0 "R2" H 5670 2546 50  0000 L CNN
 F 1 "33k" H 5670 2455 50  0000 L CNN
-F 2 "" V 5530 2500 50  0001 C CNN
+F 2 "Resistors_SMD:R_0603" V 5530 2500 50  0001 C CNN
 F 3 "~" H 5600 2500 50  0001 C CNN
 	1    5600 2500
@@
 $EndComp
 $Comp
-L Device:R R18
+L Device:R R6
 U 1 1 616C50D0
 P 6000 2500
-F 0 "R18" H 6070 2546 50  0000 L CNN
+F 0 "R6" H 6070 2546 50  0000 L CNN
 F 1 "33k" H 6070 2455 50  0000 L CNN
-F 2 "" V 5930 2500 50  0001 C CNN
+F 2 "Resistors_SMD:R_0603" V 5930 2500 50  0001 C CNN
 F 3 "~" H 6000 2500 50  0001 C CNN
 	1    6000 2500
@@
 F 0 "L2" V 5040 3800 50  0000 C CNN
 F 1 "100uH" V 4949 3800 50  0000 C CNN
-F 2 "" H 4850 3800 50  0001 C CNN
+F 2 "Inductors_SMD:L_7.3x7.3_H3.5" H 4850 3800 50  0001 C CNN
 F 3 "~" H 4850 3800 50  0001 C CNN
 	1    4850 3800
@@
 $EndComp
 $Comp
-L Device:L L3
+L Device:L L1
 U 1 1 616C673A
 P 4750 2300
-F 0 "L3" V 4940 2300 50  0000 C CNN
+F 0 "L1" V 4940 2300 50  0000 C CNN
 F 1 "100uH" V 4849 2300 50  0000 C CNN
-F 2 "" H 4750 2300 50  0001 C CNN
+F 2 "Inductors_SMD:L_7.3x7.3_H3.5" H 4750 2300 50  0001 C CNN
 F 3 "~" H 4750 2300 50  0001 C CNN
 	1    4750 2300
@@
 $EndComp
 $Comp
-L Device:C C17
+L Device:C C6
 U 1 1 616C7552
 P 5100 2500
-F 0 "C17" H 5215 2546 50  0000 L CNN
+F 0 "C6" H 5215 2546 50  0000 L CNN
 F 1 "33nF" H 5215 2455 50  0000 L CNN
-F 2 "" H 5138 2350 50  0001 C CNN
+F 2 "Capacitors_SMD:C_0603" H 5138 2350 50  0001 C CNN
 F 3 "~" H 5100 2500 50  0001 C CNN
 	1    5100 2500
@@
 $EndComp
 $Comp
-L Device:C C15
+L Device:C C7
 U 1 1 616C7F4E
 P 5200 4100
-F 0 "C15" H 5315 4146 50  0000 L CNN
+F 0 "C7" H 5315 4146 50  0000 L CNN
 F 1 "33nF" H 5315 4055 50  0000 L CNN
-F 2 "" H 5238 3950 50  0001 C CNN
+F 2 "Capacitors_SMD:C_0603" H 5238 3950 50  0001 C CNN
 F 3 "~" H 5200 4100 50  0001 C CNN
 	1    5200 4100
@@
 $EndComp
 $Comp
-L Device:CP C14
+L Device:CP C9
 U 1 1 616C8E66
 P 6750 4350
-F 0 "C14" H 6868 4396 50  0000 L CNN
+F 0 "C9" H 6868 4396 50  0000 L CNN
 F 1 "100uF" H 6868 4305 50  0000 L CNN
-F 2 "" H 6788 4200 50  0001 C CNN
+F 2 "Capacitors_SMD:CP_Elec_5x4.5" H 6788 4200 50  0001 C CNN
 F 3 "~" H 6750 4350 50  0001 C CNN
 	1    6750 4350
@@
 $EndComp
 $Comp
-L Device:CP C16
+L Device:CP C8
 U 1 1 616C9D51
 P 6600 2650
-F 0 "C16" H 6718 2696 50  0000 L CNN
+F 0 "C8" H 6718 2696 50  0000 L CNN
 F 1 "100uF" H 6718 2605 50  0000 L CNN
-F 2 "" H 6638 2500 50  0001 C CNN
+F 2 "Capacitors_SMD:CP_Elec_5x4.5" H 6638 2500 50  0001 C CNN
 F 3 "~" H 6600 2650 50  0001 C CNN
 	1    6600 2650
@@
 $EndComp
 $Comp
-L Device:CP C5
+L Device:CP C10
 U 1 1 616CA9C1
 P 7350 4350
-F 0 "C5" H 7468 4396 50  0000 L CNN
+F 0 "C10" H 7468 4396 50  0000 L CNN
 F 1 "4.7uF" H 7468 4305 50  0000 L CNN
-F 2 "" H 7388 4200 50  0001 C CNN
+F 2 "Capacitors_SMD:CP_Elec_3x5.3" H 7388 4200 50  0001 C CNN
 F 3 "~" H 7350 4350 50  0001 C CNN
 	1    7350 4350
@@
 $EndComp
 $Comp
-L Device:CP C18
+L Device:CP C5
 U 1 1 616CB0D0
 P 2600 4300
-F 0 "C18" H 2718 4346 50  0000 L CNN
+F 0 "C5" H 2718 4346 50  0000 L CNN
 F 1 "47uF" H 2718 4255 50  0000 L CNN
-F 2 "" H 2638 4150 50  0001 C CNN
+F 2 "Capacitors_SMD:CP_Elec_5x4.5" H 2638 4150 50  0001 C CNN
 F 3 "~" H 2600 4300 50  0001 C CNN
 	1    2600 4300
@@
 $EndComp
 $Comp
-L Device:CP C6
+L Device:CP C11
 U 1 1 616CBAF5
 P 8950 4250
-F 0 "C6" H 9068 4296 50  0000 L CNN
+F 0 "C11" H 9068 4296 50  0000 L CNN
 F 1 "4.7uF" H 9068 4205 50  0000 L CNN
-F 2 "" H 8988 4100 50  0001 C CNN
+F 2 "Capacitors_SMD:CP_Elec_3x5.3" H 8988 4100 50  0001 C CNN
 F 3 "~" H 8950 4250 50  0001 C CNN
 	1    8950 4250
@@
 $EndComp
 $Comp
-L Regulator_Linear:AMS1117-5.0 U?
+L Regulator_Linear:AMS1117-5.0 U4
 U 1 1 616CCBF8
 P 8200 3800
-F 0 "U?" H 8200 4042 50  0000 C CNN
+F 0 "U4" H 8200 4042 50  0000 C CNN
 F 1 "AMS1117-5.0" H 8200 3951 50  0000 C CNN
-F 2 "Package_TO_SOT_SMD:SOT-223-3_TabPin2" H 8200 4000 50  0001 C CNN
+F 2 "TO_SOT_Packages_SMD:SOT-223-3_TabPin2" H 8200 4000 50  0001 C CNN
 F 3 "http://www.advanced-monolithic.com/pdf/ds1117.pdf" H 8300 3550 50  0001 C CNN
 	1    8200 3800
@@
 $EndComp
 $Comp
-L Device:D_Schottky D5
+L Device:D_Schottky D1
 U 1 1 616D1421
 P 4550 4650
-F 0 "D5" V 4504 4730 50  0000 L CNN
+F 0 "D1" V 4504 4730 50  0000 L CNN
 F 1 "5S310" V 4595 4730 50  0000 L CNN
-F 2 "" H 4550 4650 50  0001 C CNN
+F 2 "Diodes_SMD:D_SOD-123" H 4550 4650 50  0001 C CNN
 F 3 "~" H 4550 4650 50  0001 C CNN
 	1    4550 4650
@@
 	5200 4400 5600 4400
 $Comp
-L Local:XL7005A U5
+L Local:XL7005A U2
 U 1 1 616E3EAE
 P 3800 4250
-F 0 "U5" H 3800 4715 50  0000 C CNN
+F 0 "U2" H 3800 4715 50  0000 C CNN
 F 1 "XL7005A" H 3800 4624 50  0000 C CNN
-F 2 "" H 3800 3900 50  0001 C CNN
+F 2 "Housings_SOIC:SOIC-8-1EP_3.9x4.9mm_Pitch1.27mm" H 3800 3900 50  0001 C CNN
 F 3 "" H 3800 3900 50  0001 C CNN
 	1    3800 4250
@@
 	2600 4450 2600 4550
 Wire Wire Line
-	2600 4950 3450 4950
+	2600 4950 3300 4950
 Connection ~ 4200 4950
 $Comp
-L power:GND #PWR?
+L power:GND #PWR010
 U 1 1 616EE13E
 P 2350 4600
-F 0 "#PWR?" H 2350 4350 50  0001 C CNN
+F 0 "#PWR010" H 2350 4350 50  0001 C CNN
 F 1 "GND" H 2355 4427 50  0000 C CNN
 F 2 "" H 2350 4600 50  0001 C CNN
@@
 Connection ~ 5600 3300
 $Comp
-L Device:D_Schottky D6
+L Device:D_Schottky D2
 U 1 1 617101C7
 P 4600 3100
-F 0 "D6" V 4554 3180 50  0000 L CNN
+F 0 "D2" V 4554 3180 50  0000 L CNN
 F 1 "5S310" V 4645 3180 50  0000 L CNN
-F 2 "" H 4600 3100 50  0001 C CNN
+F 2 "Diodes_SMD:D_SOD-123" H 4600 3100 50  0001 C CNN
 F 3 "~" H 4600 3100 50  0001 C CNN
 	1    4600 3100
@@
 	5100 2650 5100 2800
 $Comp
-L Local:XL7005A U6
+L Local:XL7005A U3
 U 1 1 6171D115
 P 3950 2700
-F 0 "U6" H 3950 3165 50  0000 C CNN
+F 0 "U3" H 3950 3165 50  0000 C CNN
 F 1 "XL7005A" H 3950 3074 50  0000 C CNN
-F 2 "" H 3950 2350 50  0001 C CNN
+F 2 "Housings_SOIC:SOIC-8-1EP_3.9x4.9mm_Pitch1.27mm" H 3950 2350 50  0001 C CNN
 F 3 "" H 3950 2350 50  0001 C CNN
 	1    3950 2700
@@
 	4300 3300 4300 2950
 Connection ~ 4600 3300
-Connection ~ 3450 4950
-Wire Wire Line
-	3450 4950 4200 4950
 Wire Wire Line
 	3450 2500 3600 2500
@@
 	4300 3300 3450 3300
 Connection ~ 4300 3300
-Connection ~ 3450 3300
 Wire Wire Line
 	3450 3300 3450 2950
@@
 	4400 2500 4300 2500
 $Comp
-L power:+3.3V #PWR?
+L power:+3.3V #PWR011
 U 1 1 617338F7
 P 8550 2300
-F 0 "#PWR?" H 8550 2150 50  0001 C CNN
+F 0 "#PWR011" H 8550 2150 50  0001 C CNN
 F 1 "+3.3V" V 8565 2428 50  0000 L CNN
 F 2 "" H 8550 2300 50  0001 C CNN
@@
 $EndComp
 $Comp
-L power:+12V #PWR?
+L power:+12V #PWR012
 U 1 1 617344C3
 P 8550 2600
-F 0 "#PWR?" H 8550 2450 50  0001 C CNN
+F 0 "#PWR012" H 8550 2450 50  0001 C CNN
 F 1 "+12V" V 8565 2728 50  0000 L CNN
 F 2 "" H 8550 2600 50  0001 C CNN
@@
 $EndComp
 $Comp
-L power:+5V #PWR?
+L power:+5V #PWR013
 U 1 1 61734DF6
 P 8600 2900
-F 0 "#PWR?" H 8600 2750 50  0001 C CNN
+F 0 "#PWR013" H 8600 2750 50  0001 C CNN
 F 1 "+5V" V 8615 3028 50  0000 L CNN
 F 2 "" H 8600 2900 50  0001 C CNN
@@
 Connection ~ 6600 2300
 Wire Wire Line
-	3450 3300 3450 4950
+	3300 3300 3300 4050
+Connection ~ 3300 4950
+Wire Wire Line
+	3300 4950 4200 4950
+Wire Wire Line
+	3300 3300 3450 3300
+Connection ~ 3450 3300
+Wire Wire Line
+	3450 4050 3300 4050
+Connection ~ 3300 4050
+Wire Wire Line
+	3300 4050 3300 4200
+Wire Wire Line
+	3450 4200 3300 4200
+Connection ~ 3300 4200
+Wire Wire Line
+	3300 4200 3300 4350
+Wire Wire Line
+	3450 4350 3300 4350
+Connection ~ 3300 4350
+Wire Wire Line
+	3300 4350 3300 4500
+Wire Wire Line
+	3450 4500 3300 4500
+Connection ~ 3300 4500
+Wire Wire Line
+	3300 4500 3300 4950
 $EndSCHEMATC
