File: interfaz.sch (KiCad schematic (older format))
At the start: 0 parts

Commit message: Esquemático acabado y asignación de huellas
Parts:
- added C25, C26, C27, C28: 0.1u, Capacitors_SMD:C_0603, symbol Device:C
- added J4: Pantalla LCD, Pin_Headers:Pin_Header_Straight_1x06_Pitch2.54mm, symbol Connector_Generic:Conn_01x06
- added J5: GSM900A, Pin_Headers:Pin_Header_Straight_1x05_Pitch2.54mm, symbol Connector_Generic:Conn_01x05
- added Q10, Q11: BSN20, TO_SOT_Packages_SMD:SOT-23, symbol Transistor_FET:BSN20
- added R37, R38, R39, R40: 10k, Resistors_SMD:R_0603, symbol Device:R
- added SW2, SW3, SW4, SW5: SW_Push, Pin_Headers:Pin_Header_Straight_1x02_Pitch2.54mm, symbol Switch:SW_Push
Connections:
- new net +3V3: J4.1 (Pin_1), Q10.1 (G), Q11.1 (G), R37.1, R39.1
- new net +5V: J5.1 (Pin_1), R38.1, R40.1
- new net BTN_0: C25.1, SW2.2
- new net BTN_1: C26.1, SW3.2
- new net BTN_2: C27.1, SW4.2
- new net BTN_3: C28.1, SW5.2
- new net GND: C25.2, C26.2, C27.2, C28.2, J4.2 (Pin_2), J5.2 (Pin_2), SW2.1, SW3.1, SW4.1, SW5.1
- new net MISO: J4.5 (Pin_5)
- new net MOSI: J4.4 (Pin_4)
- new net SCK: J4.3 (Pin_3)
- new net UART5_RX: J5.5 (Pin_5), Q10.3 (D), R38.2
- new net UART5_TX: J5.4 (Pin_4), Q11.3 (D), R40.2
- new net UART_INT: J5.3 (Pin_3)
- new net UART_RX: Q10.2 (S), R37.2
- new net UART_TX: Q11.2 (S), R39.2
- new net ~SS0: J4.6 (Pin_6)
