File: MPPT.sch (KiCad schematic (older format))
At the start: 0 parts

Commit message: Trabajo de Carmen y Javi
Parts:
- added Battery_1: 0-50V, symbol Device:Battery
- added C1, C2, C3, C5, C8: 100nF, symbol Device:C
- added C4, C7: 470uF, symbol Device:CP
- added C6: 10uF, symbol Device:CP
- added D1: LED, symbol Device:LED
- added D2, D6: 1N4007, Diode_THT:D_DO-41_SOD81_P10.16mm_Horizontal, symbol Diode:1N4007
- added D3, D4, D5: SS310, symbol Device:D_Schottky
- added F1, F2: 35A, symbol Device:Fuse
- added L1: 60uH, symbol Device:L
- added Pin_header_P-2.54mm_1: B1212S-1W, symbol Connector:Conn_01x04_Female
- added Q1, Q2, Q3, Q4: CSD19505, Package_TO_SOT_SMD:TDSON-8-1, symbol Transistor_FET:CSD19502Q5B
- added R1, R2, R5, R6, R7: 10K, symbol Device:R
- added R10, R8: 100, symbol Device:R
- added R11, R9: 100K, symbol Device:R
- added R12, R13: 47K, symbol Device:R
- added R14: 1K, symbol Device:R
- added R3: 200K, symbol Device:R
- added R4: 5.1K, symbol Device:R
- added Solar_Panel_1: 15-80V, symbol Device:Battery
- added U1: IR2104, symbol Driver_FET:IR2104
Connections:
- net labels added: +12V, A1, A3, BCCU, GND, IR2104-EN, IR2104-IN, XL7005A_VIN
- wire segments 0 -> 159

Commit message: Esquemático acabado y asignación de huellas
Parts:
- removed Pin_header_P-2.54mm_1: B1212S-1W, symbol Connector:Conn_01x04_Female
- removed Q1, Q2, Q3, Q4: CSD19505, Package_TO_SOT_SMD:TDSON-8-1, symbol Transistor_FET:CSD19502Q5B
- added J8: B1212S-1W, Pin_Headers:Pin_Header_Straight_1x04_Pitch2.54mm, symbol Connector_Generic:Conn_01x04
- added Q1, Q2, Q3, Q4: CSD19505, TO_SOT_Packages_THT:TO-220-3_Vertical, symbol Device:Q_NMOS_GDS
- C12: renamed from C3; footprint (none) -> Capacitors_SMD:C_0603
- C13: renamed from C4; footprint (none) -> Capacitors_SMD:CP_Elec_6.3x4.5
- C14: renamed from C5; footprint (none) -> Capacitors_SMD:C_0603
- C15: renamed from C1; footprint (none) -> Capacitors_SMD:C_0603
- C16: renamed from C6; footprint (none) -> Capacitors_SMD:CP_Elec_3x5.3
- C17: renamed from C2; footprint (none) -> Capacitors_SMD:C_0603
- C18: renamed from C7; footprint (none) -> Capacitors_SMD:CP_Elec_6.3x4.5
- C19: renamed from C8; footprint (none) -> Capacitors_SMD:C_0603
- D3: renamed from D2; footprint Diode_THT:D_DO-41_SOD81_P10.16mm_Horizontal -> Diodes_SMD:D_SOD-123
- D4: renamed from D1; footprint (none) -> Diodes_SMD:D_0603
- D5: renamed from D3; footprint (none) -> Diodes_SMD:D_SOD-123
- D6: renamed from D5; footprint (none) -> Diodes_SMD:D_SOD-123
- D7: renamed from D4; footprint (none) -> Diodes_SMD:D_SOD-123
- D8: renamed from D6; footprint Diode_THT:D_DO-41_SOD81_P10.16mm_Horizontal -> Diodes_SMD:D_SOD-123
- F1, F2: footprint (none) -> Fuse_Holders_and_Fuses:Fuseholder5x20_horiz_SemiClosed_Casing10x25mm
- J6: renamed from Solar_Panel_1; footprint (none) -> Connectors:Banana_Jack_2Pin
- J7: renamed from Battery_1; footprint (none) -> Connectors:Banana_Jack_2Pin
- L3: renamed from L1; footprint (none) -> Inductors_SMD:L_6.3x6.3_H3
- R10: renamed from R5; footprint (none) -> Resistors_SMD:R_0603
- R11: renamed from R6; footprint (none) -> Resistors_SMD:R_0603
- R12: renamed from R2; footprint (none) -> Resistors_SMD:R_0603
- R13: renamed from R1; footprint (none) -> Resistors_SMD:R_0603
- R14: renamed from R10; footprint (none) -> Resistors_SMD:R_0603
- R15: renamed from R8; footprint (none) -> Resistors_SMD:R_0603
- R16: renamed from R9; footprint (none) -> Resistors_SMD:R_0603
- R17: renamed from R11; footprint (none) -> Resistors_SMD:R_0603
- R18: renamed from R7; footprint (none) -> Resistors_SMD:R_0603
- R19: renamed from R12; footprint (none) -> Resistors_SMD:R_0603
- R20: renamed from R14; footprint (none) -> Resistors_SMD:R_0603
- R21: renamed from R13; footprint (none) -> Resistors_SMD:R_0603
- R8: renamed from R3; footprint (none) -> Resistors_SMD:R_0603
- R9: renamed from R4; footprint (none) -> Resistors_SMD:R_0603
- U5: renamed from U1; footprint (none) -> Housings_SOIC:SOIC-8_3.9x4.9mm_Pitch1.27mm

Commit message: Modelos 3D dificiles incluidos
Parts:
- F1, F2: footprint Fuse_Holders_and_Fuses:Fuseholder5x20_horiz_SemiClosed_Casing10x25mm -> Fuse_Holders_and_Fuses:BladeFuse-CarType
- J6, J7: footprint Connectors:Banana_Jack_2Pin -> Wire_Pads:SolderWirePad_2x_1-5mmDrill
- L3: footprint Inductors_SMD:L_6.3x6.3_H3 -> Inductors_THT:L_Toroid_Vertical_L28.6mm_W14.3mm_P11.43mm_Bourns_5700
Changed lines of the file:
@@
 F 0 "L3" V 8540 4420 50  0000 C CNN
 F 1 "60uH" V 8449 4420 50  0000 C CNN
-F 2 "Inductors_SMD:L_6.3x6.3_H3" H 8350 4420 50  0001 C CNN
+F 2 "Inductors_THT:L_Toroid_Vertical_L28.6mm_W14.3mm_P11.43mm_Bourns_5700" H 8350 4420 50  0001 C CNN
 F 3 "~" H 8350 4420 50  0001 C CNN
 	1    8350 4420
@@
 F 0 "F2" V 9863 4420 50  0000 C CNN
 F 1 "35A" V 9954 4420 50  0000 C CNN
-F 2 "Fuse_Holders_and_Fuses:Fuseholder5x20_horiz_SemiClosed_Casing10x25mm" V 9990 4420 50  0001 C CNN
+F 2 "Fuse_Holders_and_Fuses:BladeFuse-CarType" V 9990 4420 50  0001 C CNN
 F 3 "~" H 10060 4420 50  0001 C CNN
 	1    10060 4420
@@
 F 0 "F1" V 1363 2460 50  0000 C CNN
 F 1 "35A" V 1454 2460 50  0000 C CNN
-F 2 "Fuse_Holders_and_Fuses:Fuseholder5x20_horiz_SemiClosed_Casing10x25mm" V 1490 2460 50  0001 C CNN
+F 2 "Fuse_Holders_and_Fuses:BladeFuse-CarType" V 1490 2460 50  0001 C CNN
 F 3 "~" H 1560 2460 50  0001 C CNN
 	1    1560 2460
@@
 F 0 "J6" H 1268 3196 50  0000 L CNN
 F 1 "15-80V" H 1268 3105 50  0000 L CNN
-F 2 "Connectors:Banana_Jack_2Pin" V 1160 3210 50  0001 C CNN
+F 2 "Wire_Pads:SolderWirePad_2x_1-5mmDrill" V 1160 3210 50  0001 C CNN
 F 3 "~" V 1160 3210 50  0001 C CNN
 	1    1160 3150
@@
 F 0 "J7" H 10598 5206 50  0000 L CNN
 F 1 "0-50V" H 10598 5115 50  0000 L CNN
-F 2 "Connectors:Banana_Jack_2Pin" V 10490 5220 50  0001 C CNN
+F 2 "Wire_Pads:SolderWirePad_2x_1-5mmDrill" V 10490 5220 50  0001 C CNN
 F 3 "~" V 10490 5220 50  0001 C CNN
 	1    10490 5160

Commit message: Punto de control pistas
Connections:
- net +BATT: now reaches D8.2 (A), F2.1, J7.1 (+)
Changed lines of the file:
@@
 L power:GND #PWR014
 U 1 1 617447C8
-P 2260 3770
+P 1940 3770
 AR Path="/61644C06/617447C8" Ref="#PWR014"  Part="1"
 AR Path="/617447C8" Ref="#PWR?"  Part="1"
-F 0 "#PWR014" H 2260 3520 50  0001 C CNN
-F 1 "GND" H 2265 3597 50  0000 C CNN
-F 2 "" H 2260 3770 50  0001 C CNN
-F 3 "" H 2260 3770 50  0001 C CNN
-	1    2260 3770
+F 0 "#PWR014" H 1940 3520 50  0001 C CNN
+F 1 "GND" H 1945 3597 50  0000 C CNN
+F 2 "" H 1940 3770 50  0001 C CNN
+F 3 "" H 1940 3770 50  0001 C CNN
+	1    1940 3770
 	1    0    0    -1
 $EndComp
@@
 	2260 3500 2260 3650
 Wire Wire Line
-	2260 3650 1860 3650
+	2260 3650 1940 3650
 Wire Wire Line
 	1860 3650 1860 3480
@@
 Connection ~ 3080 3310
 Wire Wire Line
-	2260 3770 2260 3650
+	1940 3770 1940 3650
 Wire Wire Line
 	1160 2140 1160 2460
@@
 	1160 2950 1160 2460
 Connection ~ 1160 2460
-Wire Wire Line
-	1160 3350 1160 3650
-Wire Wire Line
-	1160 3650 1860 3650
-Connection ~ 1860 3650
 Wire Wire Line
 	8680 5080 8680 5850
@@
 	6320 2800 6320 2610
 $Comp
+L Device:Battery J7
+U 1 1 61744799
+P 10490 5160
+AR Path="/61644C06/61744799" Ref="J7"  Part="1"
+AR Path="/61744799" Ref="Battery_?"  Part="1"
+F 0 "J7" H 10598 5206 50  0000 L CNN
+F 1 "0-50V" H 10598 5115 50  0000 L CNN
+F 2 "Wire_Pads:SolderWirePad_2x_1-5mmDrill" V 10490 5220 50  0001 C CNN
+F 3 "~" V 10490 5220 50  0001 C CNN
+	1    10490 5160
+	1    0    0    -1
+$EndComp
+$Comp
+L Connector_Generic:Conn_01x04 J8
+U 1 1 61D0BDE9
+P 5850 950
+F 0 "J8" V 5814 662 50  0000 R CNN
+F 1 "B1212S-1W" V 5723 662 50  0000 R CNN
+F 2 "Pin_Headers:Pin_Header_Straight_1x04_Pitch2.54mm" H 5850 950 50  0001 C CNN
+F 3 "~" H 5850 950 50  0001 C CNN
+	1    5850 950
+	0    -1   -1   0
+$EndComp
+Wire Wire Line
+	5750 1150 5750 1440
+Wire Wire Line
+	5850 1150 5850 1670
+Wire Wire Line
+	5760 1670 5850 1670
+Wire Wire Line
+	6050 1150 6050 1500
+Wire Wire Line
+	5950 1150 5950 1890
+Wire Wire Line
+	5950 1890 6050 1890
+Wire Wire Line
+	5950 2800 6320 2800
+$Comp
+L Device:Q_NMOS_GDS Q2
+U 1 1 61E1C7AE
+P 6980 2190
+F 0 "Q2" H 7185 2144 50  0000 L CNN
+F 1 "CSD19505" H 7185 2235 50  0000 L CNN
+F 2 "TO_SOT_Packages_THT:TO-220-3_Vertical" H 7180 2290 50  0001 C CNN
+F 3 "~" H 6980 2190 50  0001 C CNN
+	1    6980 2190
+	-1   0    0    1
+$EndComp
+$Comp
+L Device:Q_NMOS_GDS Q1
+U 1 1 61E52C62
+P 5230 2360
+F 0 "Q1" V 5479 2360 50  0000 C CNN
+F 1 "CSD19505" V 5570 2360 50  0000 C CNN
+F 2 "TO_SOT_Packages_THT:TO-220-3_Vertical" H 5430 2460 50  0001 C CNN
+F 3 "~" H 5230 2360 50  0001 C CNN
+	1    5230 2360
+	0    1    1    0
+$EndComp
+$Comp
+L Device:Q_NMOS_GDS Q3
+U 1 1 61E85D64
+P 7600 3410
+F 0 "Q3" H 7804 3456 50  0000 L CNN
+F 1 "CSD19505" H 7804 3365 50  0000 L CNN
+F 2 "TO_SOT_Packages_THT:TO-220-3_Vertical" H 7800 3510 50  0001 C CNN
+F 3 "~" H 7600 3410 50  0001 C CNN
+	1    7600 3410
+	1    0    0    -1
+$EndComp
+$Comp
+L Device:Q_NMOS_GDS Q4
+U 1 1 61EA5566
+P 7600 5240
+F 0 "Q4" H 7804 5286 50  0000 L CNN
+F 1 "CSD19505" H 7804 5195 50  0000 L CNN
+F 2 "TO_SOT_Packages_THT:TO-220-3_Vertical" H 7800 5340 50  0001 C CNN
+F 3 "~" H 7600 5240 50  0001 C CNN
+	1    7600 5240
+	1    0    0    -1
+$EndComp
+Connection ~ 1940 3650
+Wire Wire Line
+	1940 3650 1860 3650
+$Comp
+L power:GND #PWR0101
+U 1 1 61CDFD8D
+P 1160 3465
+AR Path="/61644C06/61CDFD8D" Ref="#PWR0101"  Part="1"
+AR Path="/61CDFD8D" Ref="#PWR?"  Part="1"
+F 0 "#PWR0101" H 1160 3215 50  0001 C CNN
+F 1 "GND" H 1165 3292 50  0000 C CNN
+F 2 "" H 1160 3465 50  0001 C CNN
+F 3 "" H 1160 3465 50  0001 C CNN
+	1    1160 3465
+	1    0    0    -1
+$EndComp
+$Comp
 L Device:Battery J6
 U 1 1 6174480B
@@
 	1    0    0    -1
 $EndComp
-$Comp
-L Device:Battery J7
-U 1 1 61744799
-P 10490 5160
-AR Path="/61644C06/61744799" Ref="J7"  Part="1"
-AR Path="/61744799" Ref="Battery_?"  Part="1"
-F 0 "J7" H 10598 5206 50  0000 L CNN
-F 1 "0-50V" H 10598 5115 50  0000 L CNN
-F 2 "Wire_Pads:SolderWirePad_2x_1-5mmDrill" V 10490 5220 50  0001 C CNN
-F 3 "~" V 10490 5220 50  0001 C CNN
-	1    10490 5160
-	1    0    0    -1
-$EndComp
-$Comp
-L Connector_Generic:Conn_01x04 J8
-U 1 1 61D0BDE9
-P 5850 950
-F 0 "J8" V 5814 662 50  0000 R CNN
-F 1 "B1212S-1W" V 5723 662 50  0000 R CNN
-F 2 "Pin_Headers:Pin_Header_Straight_1x04_Pitch2.54mm" H 5850 950 50  0001 C CNN
-F 3 "~" H 5850 950 50  0001 C CNN
-	1    5850 950
-	0    -1   -1   0
-$EndComp
-Wire Wire Line
-	5750 1150 5750 1440
-Wire Wire Line
-	5850 1150 5850 1670
-Wire Wire Line
-	5760 1670 5850 1670
-Wire Wire Line
-	6050 1150 6050 1500
-Wire Wire Line
-	5950 1150 5950 1890
-Wire Wire Line
-	5950 1890 6050 1890
-Wire Wire Line
-	5950 2800 6320 2800
-$Comp
-L Device:Q_NMOS_GDS Q2
-U 1 1 61E1C7AE
-P 6980 2190
-F 0 "Q2" H 7185 2144 50  0000 L CNN
-F 1 "CSD19505" H 7185 2235 50  0000 L CNN
-F 2 "TO_SOT_Packages_THT:TO-220-3_Vertical" H 7180 2290 50  0001 C CNN
-F 3 "~" H 6980 2190 50  0001 C CNN
-	1    6980 2190
-	-1   0    0    1
-$EndComp
-$Comp
-L Device:Q_NMOS_GDS Q1
-U 1 1 61E52C62
-P 5230 2360
-F 0 "Q1" V 5479 2360 50  0000 C CNN
-F 1 "CSD19505" V 5570 2360 50  0000 C CNN
-F 2 "TO_SOT_Packages_THT:TO-220-3_Vertical" H 5430 2460 50  0001 C CNN
-F 3 "~" H 5230 2360 50  0001 C CNN
-	1    5230 2360
-	0    1    1    0
-$EndComp
-$Comp
-L Device:Q_NMOS_GDS Q3
-U 1 1 61E85D64
-P 7600 3410
-F 0 "Q3" H 7804 3456 50  0000 L CNN
-F 1 "CSD19505" H 7804 3365 50  0000 L CNN
-F 2 "TO_SOT_Packages_THT:TO-220-3_Vertical" H 7800 3510 50  0001 C CNN
-F 3 "~" H 7600 3410 50  0001 C CNN
-	1    7600 3410
-	1    0    0    -1
-$EndComp
-$Comp
-L Device:Q_NMOS_GDS Q4
-U 1 1 61EA5566
-P 7600 5240
-F 0 "Q4" H 7804 5286 50  0000 L CNN
-F 1 "CSD19505" H 7804 5195 50  0000 L CNN
-F 2 "TO_SOT_Packages_THT:TO-220-3_Vertical" H 7800 5340 50  0001 C CNN
-F 3 "~" H 7600 5240 50  0001 C CNN
-	1    7600 5240
-	1    0    0    -1
-$EndComp
+Wire Wire Line
+	1160 3465 1160 3350
+$Comp
+L power:+BATT #PWR?
+U 1 1 61D3F9DC
+P 10900 4350
+F 0 "#PWR?" H 10900 4200 50  0001 C CNN
+F 1 "+BATT" H 10915 4523 50  0000 C CNN
+F 2 "" H 10900 4350 50  0001 C CNN
+F 3 "" H 10900 4350 50  0001 C CNN
+	1    10900 4350
+	1    0    0    -1
+$EndComp
+Wire Wire Line
+	10490 4420 10900 4420
+Wire Wire Line
+	10900 4420 10900 4350
 $EndSCHEMATC
