File: inverter.sch (KiCad schematic (older format))
At the start: 31 parts, among them J2 Conn_01x17, J3 FAN, J9 AC, Q5 BSN20, Q6 IRF3205, Q7 IRF3205, Q8 IRF3205, Q9 IRF3205, T1 Transformer_1P_1S

Commit message: Modelos 3D dificiles incluidos
Parts:
- J9: footprint Connectors:Banana_Jack_2Pin -> Wire_Pads:SolderWirePad_2x_1-5mmDrill
Changed lines of the file:
@@
 F 0 "J9" H 9880 5342 50  0000 L CNN
 F 1 "AC" H 9880 5251 50  0000 L CNN
-F 2 "Connectors:Banana_Jack_2Pin" H 9800 5350 50  0001 C CNN
+F 2 "Wire_Pads:SolderWirePad_2x_1-5mmDrill" H 9800 5350 50  0001 C CNN
 F 3 "~" H 9800 5350 50  0001 C CNN
 	1    9800 5350

Commit message: Punto de control pistas
Connections:
- net +12V: no longer Q6.2 (D), Q8.2 (D)
- new net +BATT: Q6.2 (D), Q8.2 (D)
Changed lines of the file:
@@
 Wire Wire Line
 	7400 2750 7400 3200
-$Comp
-L power:+12V #PWR030
-U 1 1 61BAE807
-P 6400 1200
-F 0 "#PWR030" H 6400 1050 50  0001 C CNN
-F 1 "+12V" H 6415 1373 50  0000 C CNN
-F 2 "" H 6400 1200 50  0001 C CNN
-F 3 "" H 6400 1200 50  0001 C CNN
-	1    6400 1200
-	1    0    0    -1
-$EndComp
 Wire Wire Line
 	6400 1200 6400 1450
@@
 Wire Wire Line
 	9600 5450 9250 5450
+$Comp
+L power:+BATT #PWR?
+U 1 1 61D3E7B8
+P 6400 1200
+F 0 "#PWR?" H 6400 1050 50  0001 C CNN
+F 1 "+BATT" H 6415 1373 50  0000 C CNN
+F 2 "" H 6400 1200 50  0001 C CNN
+F 3 "" H 6400 1200 50  0001 C CNN
+	1    6400 1200
+	1    0    0    -1
+$EndComp
 $EndSCHEMATC
