File: proyectoSolar.kicad_pcb (KiCad board)
At the start: 2 copper layers, 124 parts, among them J1 UART/PROG, J2 Conn_01x17, J3 FAN, J4 Pantalla LCD, J5 GSM900A, J6 15-80V, J7 0-50V, J8 B1212S-1W, J9 AC, Q1 CSD19505, Q10 BSN20, Q11 BSN20, Q2 CSD19505, Q3 CSD19505, Q4 CSD19505, Q5 BSN20, Q6 IRF3205, Q7 IRF3205, Q8 IRF3205, Q9 IRF3205, SW1 SW_Push, SW2 SW_Push, SW3 SW_Push, SW4 SW_Push, SW5 SW_Push, T1 Transformer_1P_1S, U1 ESP32-WROOM-32D, U2 XL7005A, U3 XL7005A, U4 AMS1117-5.0, U5 IR2104, U6 ACS712xLCTR-20A, U7 ADS1015IDGS

Commit message: Punto restauracion 18:29
Parts:
- C6: footprint Capacitors_SMD:C_0603 -> Capacitors_SMD:CP_Elec_3x5.3
- moved J2 275.9 mm to (144.0, 83.8), turned to 90 degrees
- moved U7 220.9 mm to (86.9, 121.5), turned to 90 degrees
- moved C12 217.7 mm to (82.5, 120.0), turned to 90 degrees
- moved R41 215.3 mm to (88.5, 116.0), turned to 90 degrees
- moved C29 212.5 mm to (85.0, 116.2), turned to 90 degrees
- moved R36 192.8 mm to (211.0, 122.8), turned to 180 degrees
- moved J1 187.8 mm to (129.5, 129.2), turned to 270 degrees
- moved R35 186.9 mm to (211.0, 117.2), turned to 180 degrees
- moved C3 183.2 mm to (164.5, 125.2), turned to 270 degrees
- moved RV1 181.3 mm to (204.0, 117.8), turned to 180 degrees
- moved C26 178.5 mm to (159.8, 92.2), turned to 270 degrees
- moved C25 178.1 mm to (162.8, 92.2), turned to 270 degrees
- moved R30 178.1 mm to (177.2, 74.2)
- moved SW3 176.0 mm to (147.0, 91.0), turned to 270 degrees
- moved C28 173.4 mm to (159.8, 95.5), turned to 270 degrees
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Connections:
- U3 pad 9: (no net) -> GND
Other:
- copper layers 2 -> 4
- net class Default: trace_width 0.25 -> 0.3

Commit message: Todo en su sitio
Parts:
- moved R25 255.0 mm to (188.2, 90.8), turned to 90 degrees
- moved R28 226.7 mm to (150.0, 73.8), turned to 180 degrees
- moved C23 215.5 mm to (197.5, 120.2), turned to 180 degrees
- moved D9 210.3 mm to (151.0, 69.5), turned to 180 degrees
- moved C22 206.0 mm to (179.5, 94.2), turned to 180 degrees
- moved R27 203.1 mm to (170.8, 71.8)
- moved R29 202.4 mm to (170.5, 73.8), turned to 180 degrees
- moved R33 201.2 mm to (191.0, 73.5), turned to 180 degrees
- moved R26 200.5 mm to (150.2, 71.8)
- moved R31 188.5 mm to (191.2, 71.8)
- moved R34 179.3 mm to (201.5, 64.2), turned to 90 degrees
- moved R32 179.0 mm to (203.2, 64.5), turned to 270 degrees
- moved TH1 178.9 mm to (178.0, 90.5), turned to 90 degrees
- moved D10 174.2 mm to (171.5, 69.5), turned to 180 degrees
- moved Q5 173.3 mm to (192.8, 90.2), turned to 90 degrees
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Other:
- board outline added: 210 x 77 mm

Commit message: Punto de control pistas
Parts:
- C6: footprint Capacitors_SMD:CP_Elec_3x5.3 -> Capacitors_SMD:C_0603
- moved R39 60.0 mm to (122.5, 132.8), turned to 180 degrees
- moved R37 48.7 mm to (126.2, 132.8), turned to 180 degrees
- moved T1 32.2 mm to (203.5, 99.5), turned to 0 degrees
- moved D8 14.7 mm to (120.5, 111.5)
- moved R30 14.1 mm to (164.8, 71.5), turned to 270 degrees
- moved R41 10.7 mm to (86.2, 126.5)
- moved Q10 9.25 mm to (182.8, 117.5)
- moved R40 7.90 mm to (177.0, 121.5)
- moved R38 6.93 mm to (184.5, 121.5)
- moved Q11 6.00 mm to (175.2, 117.5)
- moved R12 4.25 mm to (70.5, 70.8), turned to 0 degrees
- moved C13 0.50 mm to (66.2, 94.0)
- moved F1 0.50 mm to (50.5, 94.0)
- moved F2 0.50 mm to (113.2, 113.2)
- moved L3 0.50 mm to (113.2, 74.0)
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Connections:
- D8 pad 2: Net-(D8-Pad2) -> +BATT
- F2 pad 1: Net-(D8-Pad2) -> +BATT
- J7 pad 1: Net-(D8-Pad2) -> +BATT
- Q6 pad 2: +12V -> +BATT
- Q8 pad 2: +12V -> +BATT
- T1 pad 1: /inverter/L -> /inverter/VS2
- T1 pad 2: /inverter/N -> /inverter/VS1
- T1 pad 3: /inverter/VS1 -> /inverter/N
- T1 pad 4: /inverter/VS2 -> /inverter/L
- U3 pad 9: GND -> (no net)
Routing:
- net /inverter/VS1: track 0.00 -> 107.3 mm, vias 0 -> 2
- net UART_RX: track 0.00 -> 98.8 mm, vias 0 -> 1
- net BCCU: track 0.00 -> 97.8 mm, vias 0 -> 4
- net IR2104-EN: track 0.00 -> 91.8 mm, vias 0 -> 4
- net UART_TX: track 0.00 -> 90.5 mm
- net XL7005A_VIN: track 0.00 -> 89.5 mm
- net /inverter/1LO: track 0.00 -> 84.5 mm
- net Net-(C16-Pad2): track 0.00 -> 81.9 mm
- net ADC-ALERT: track 0.00 -> 81.7 mm, vias 0 -> 4
- net A2: track 0.00 -> 67.9 mm, vias 0 -> 2
- net /inverter/IFB: track 0.00 -> 67.1 mm, vias 0 -> 1
- net /inverter/N: track 0.00 -> 65.8 mm
- net /MPPT/currentSensor/IP-: track 0.00 -> 61.9 mm
- net MISO: track 0.00 -> 61.5 mm, vias 0 -> 1
- net SDA: track 0.00 -> 56.7 mm
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- added copper zone on B.Cu, net +BATT
- added copper zone on F.Cu, net +BATT
- added copper zone on B.Cu, net /MPPT/currentSensor/IP+
- added copper zone on F.Cu, net /MPPT/currentSensor/IP+
- added copper zone on In1.Cu, net /MPPT/currentSensor/IP+
- added copper zone on In2.Cu, net /MPPT/currentSensor/IP+
- added copper zone on F.Cu, net /MPPT/currentSensor/IP-
- added copper zone on In1.Cu, net /inverter/IFB
- added copper zone on B.Cu, net /inverter/VS1
- added copper zone on B.Cu, net /inverter/VS2
- added copper zone on F.Cu, net Net-(C16-Pad2)
- added copper zone on F.Cu, net Net-(C18-Pad1)
- added copper zone on B.Cu, net Net-(D3-Pad2)
- added copper zone on F.Cu, net Net-(D3-Pad2)
- added copper zone on In1.Cu, net Net-(D3-Pad2)
- added copper zone on In2.Cu, net Net-(D3-Pad2)
- added copper zone on F.Cu, net Net-(Q1-Pad2)

Commit message: Punto de control pistas
Routing:
- net +5V: track 10.9 -> 245.0 mm, vias 0 -> 4
- net +3V3: track 16.9 -> 208.5 mm, vias 0 -> 5
- net +12V: track 22.7 -> 205.2 mm, vias 0 -> 6
- net A3: track 15.3 -> 88.4 mm
- net BTN_2: track 8.31 -> 24.1 mm
- net Net-(C7-Pad2): track 12.7 -> 24.6 mm, vias 2 -> 3
- net UART_RX: track 98.8 -> 96.7 mm
- net /inverter/1HO: track 54.5 -> 55.7 mm
- net GND: vias 0 -> 55
- added copper zone on B.Cu, net GND
- added copper zone on F.Cu, net GND
- added copper zone on In1.Cu, net GND

Commit message: Acabado
Parts:
- added REF**: MountingHole_3.2mm_M3_Pad_Via, Mounting_Holes:MountingHole_3.2mm_M3_Pad_Via, F.Cu at (50.0, 67.0)
- added REF**: MountingHole_3.2mm_M3_Pad_Via, Mounting_Holes:MountingHole_3.2mm_M3_Pad_Via, F.Cu at (50.0, 132.0)
- added REF**: MountingHole_3.2mm_M3_Pad_Via, Mounting_Holes:MountingHole_3.2mm_M3_Pad_Via, F.Cu at (250.0, 132.0)
- added REF**: MountingHole_3.2mm_M3_Pad_Via, Mounting_Holes:MountingHole_3.2mm_M3_Pad_Via, F.Cu at (250.0, 67.0)
- moved C1 11.0 mm to (174.5, 113.8)
- moved C10 11.0 mm to (82.2, 112.0)
- moved C11 11.0 mm to (84.0, 128.5)
- moved C12 11.0 mm to (93.5, 120.0)
- moved C13 11.0 mm to (77.2, 94.0)
- moved C14 11.0 mm to (92.5, 109.2)
- moved C15 11.0 mm to (73.2, 106.5)
- moved C16 11.0 mm to (89.0, 102.0)
- moved C17 11.0 mm to (78.8, 106.5)
- moved C18 11.0 mm to (111.2, 102.5)
- moved C19 11.0 mm to (93.5, 123.2)
- moved C2 11.0 mm to (173.8, 110.0)
- moved C20 11.0 mm to (62.1, 82.9)
- moved C21 11.0 mm to (71.1, 77.6)
- moved C22 11.0 mm to (190.5, 94.2)
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Connections:
- U2 pad 9: (no net) -> GND
- U3 pad 9: (no net) -> GND
Routing:
- net GND: track 0.00 -> 4.46 mm, vias 55 -> 87
- net +3V3: track 208.5 -> 212.1 mm
- net Net-(C17-Pad1): track 51.1 -> 52.5 mm
- added copper zone on In2.Cu, net GND
